Commit message: Got the keyboard teleopration tool to work with scorbot, changed urdf to modify effort limits

File: scorbot_description/scorbot.urdf (robot description, URDF)
Before this commit: robot scorbot, 8 links, 7 joints
Joints:
- joint base_to_body: limit lower=-2.70526 upper=2.70526 effort=1.0 velocity=2 -> lower=-2.70526 upper=2.70526 effort=255.0 velocity=2
- joint body_to_upper_arm: limit lower=-2.26893 upper=0.610865 effort=1.0 velocity=2 -> lower=-2.26893 upper=0.610865 effort=255.0 velocity=2
- joint fore_arm_to_wrist_x: limit lower=-2.26893 upper=2.26893 effort=1.0 velocity=2 -> lower=-2.26893 upper=2.26893 effort=255.0 velocity=2
- joint upper_arm_to_fore_arm: limit lower=-2.26893 upper=2.26893 effort=1.0 velocity=2 -> lower=-2.26893 upper=2.26893 effort=255.0 velocity=2
- joint wrist_x_to_wrist_z: limit lower=-3.14 upper=3.14 effort=1.0 velocity=2 -> lower=-3.14 upper=3.14 effort=255.0 velocity=2
- joint wrist_z_to_gripper_left: limit lower=-1.13446 upper=1.13446 effort=1.0 velocity=2 -> lower=-1.13446 upper=1.13446 effort=255.0 velocity=2
- joint wrist_z_to_gripper_right: limit lower=-1.13446 upper=1.13446 effort=1.0 velocity=2 -> lower=-1.13446 upper=1.13446 effort=255.0 velocity=2
